File: ECET 318/ECET_318_Project/ECET_318_Project.kicad_pcb (KiCad board)
At the start: 2 copper layers, 87 parts, among them J1 Screw_Terminal_01x02, J2 Screw_Terminal_01x03, J3 Screw_Terminal_01x02, Q1 2N3819, U1 INA128, U10 TL082, U2 TL084, U3 TL081, U4 TL084, U6 TL081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

Commit message: Mostly finished Layout and change U5 to TL084
Parts:
- removed C22: Cdec6, Capacitor_THT:C_Disc_D3.0mm_W1.6mm_P2.50mm
- removed C23: Cdec5, Capacitor_THT:C_Disc_D3.0mm_W1.6mm_P2.50mm
- removed C24: Cdec7, Capacitor_THT:C_Disc_D3.0mm_W1.6mm_P2.50mm
- removed C25: Cdec8, Capacitor_THT:C_Disc_D3.0mm_W1.6mm_P2.50mm
- removed C26: Cdec3, Capacitor_THT:C_Disc_D3.0mm_W1.6mm_P2.50mm
- removed C27: Cdec4, Capacitor_THT:C_Disc_D3.0mm_W1.6mm_P2.50mm
- removed U6, U7, U8: TL081, Package_DIP:CERDIP-8_W7.62mm_SideBrazed_LongPads_Socket
- added C30: Cdec6, Capacitor_THT:C_Disc_D3.0mm_W1.6mm_P2.50mm, F.Cu at (224.5, 104.4)
- added C31: Cdec5, Capacitor_THT:C_Disc_D3.0mm_W1.6mm_P2.50mm, F.Cu at (241.8, 104.4)
- added U5: TL084, Package_DIP:CERDIP-14_W7.62mm_SideBrazed_LongPads_Socket, F.Cu at (229.2, 96.7)
- C21: footprint Capacitor_THT:CP_Radial_D10.0mm_P5.00mm -> Capacitor_THT:C_Disc_D3.0mm_W1.6mm_P2.50mm
- D1: footprint Diode_THT:D_5W_P12.70mm_Horizontal -> Diode_THT:D_DO-34_SOD68_P7.62mm_Horizontal
- moved Q1 213.6 mm to (207.2, 114.9)
- moved R28 193.7 mm to (196.8, 101.8)
- moved R32 192.7 mm to (196.8, 108.2)
- moved R29 192.7 mm to (196.8, 95.7)
- moved J5 191.5 mm to (185.6, 99.0), turned to -90 degrees
- moved C21 190.0 mm to (220.2, 112.2), turned to -90 degrees
- moved J4 188.0 mm to (185.6, 96.3), turned to -90 degrees
- moved D1 181.2 mm to (229.2, 118.4)
- moved R31 180.0 mm to (210.0, 108.2)
- moved R30 179.8 mm to (210.0, 101.8)
- moved R33 178.8 mm to (210.2, 95.7)
- moved R34 169.0 mm to (220.3, 89.4), turned to 180 degrees
- moved R35 161.7 mm to (227.9, 89.4)
- moved U9 159.1 mm to (193.7, 71.2)
- moved R36 148.4 mm to (241.8, 89.4), turned to -90 degrees
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Connections:
- J3 pad 1: /Peak Limiter/Peak_Limit_Out+ -> /Peak Limiter/Peak_Limit_Out-
- J3 pad 2: /Peak Limiter/Peak_Limit_Out- -> /Peak Limiter/Peak_Limit_Out+
- J4 pad 1: /Shelving_Filter_Out -> Net-(J4-Pin_1)
- J5 pad 1: Net-(J5-Pin_1) -> Net-(J4-Pin_1)
- J5 pad 2: Net-(J5-Pin_1) -> /Shelving Filter/Shelving_Filter_Out
- R13 pad 2: /Shelving Filter/Shelving_Filter_out -> /Shelving Filter/Shelving_Filter_Out
- U3 pad 6: /Shelving Filter/Shelving_Filter_out -> /Shelving Filter/Shelving_Filter_Out
Routing:
- net /Mic Amp/Mic_Amp_Out: track 0.00 -> 149.4 mm, vias 0 -> 3
- net /Peak Limiter/Peak_Limit_Out+: track 0.00 -> 60.4 mm
- net Net-(U2C--): track 0.00 -> 52.7 mm
- net Net-(U3A--): track 0.00 -> 50.3 mm
- net -15V: track 35.7 -> 74.3 mm
- net Net-(R11-Pad2): track 0.00 -> 33.5 mm
- net Net-(U2D--): track 0.00 -> 33.1 mm
- net /Peak Limiter/Peak_Limit_Out-: track 0.00 -> 29.6 mm
- net Net-(U5C--): track 0.00 -> 27.3 mm
- net Net-(D1-K): track 0.00 -> 27.3 mm
- net Net-(U5A--): track 0.00 -> 26.8 mm
- net Net-(Q1-S): track 0.00 -> 26.5 mm
- net /Shelving Filter/Shelving_Filter_Out: track 0.00 -> 21.3 mm
- net Net-(C5-Pad2): track 0.00 -> 20.0 mm
- net +15V: track 68.6 -> 88.2 mm
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Other:
- board outline added: 190 x 91 mm

Commit message: Roughly finished component placeament and routing
Parts:
- removed U9: ~, Custom_parts:BreadBoard Space
- added TP1: TestPoint_Flag, TestPoint:TestPoint_Pad_D1.5mm, F.Cu at (1.27, 1.27)
- added U6: ~, Custom_parts:800CSP1B6M2QE, F.Cu at (192.5, 104.0)
- moved J4 15.2 mm to (172.3, 103.7)
- moved J5 15.2 mm to (172.3, 106.3)
- moved C21 2.63 mm to (222.9, 111.9)
- moved C30 2.63 mm to (227.1, 104.2)
- moved C31 2.63 mm to (244.4, 104.2)
- moved D1 2.63 mm to (231.8, 118.2)
- moved Q1 2.63 mm to (209.9, 114.7)
- moved R29 2.63 mm to (199.5, 95.4)
- moved R31 2.63 mm to (212.6, 107.9)
- moved R32 2.63 mm to (199.5, 107.9)
- moved R33 2.63 mm to (212.8, 95.4)
- moved R34 2.63 mm to (223.0, 89.2)
- moved R35 2.63 mm to (230.5, 89.2)
- moved J3 2.63 mm to (254.0, 98.0)
- moved R28 2.63 mm to (199.5, 101.6)
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Routing:
- net -15V: track 74.3 -> 428.7 mm, vias 0 -> 7
- net +15V: track 88.2 -> 439.9 mm, vias 0 -> 5
- net /State Variable/State_Variable_Out: track 12.4 -> 68.7 mm, vias 0 -> 2
- net /Mic Amp/Mic_Amp_Out: track 149.4 -> 197.6 mm
- net Net-(J4-Pin_1): track 0.00 -> 23.0 mm
- net /Shelving Filter/Shelving_Filter_Out: track 21.3 -> 36.8 mm
- net /Peak Limiter/Peak_Limit_in: track 0.00 -> 7.96 mm
- net Net-(Q1-S): track 26.5 -> 27.3 mm
- added copper zone on B.Cu, net GND
- added copper zone on F.Cu, net GND
Other:
- board size 190 x 91 mm -> 191 x 86.2 mm
- board text added: "Shelving Filter"
- board text added: "State Variable"

Commit message: Added Breadboard Space and Test Points
Parts:
- added J10: Conn_01x01_Socket, TestPoint:TestPoint_THTPad_D1.5mm_Drill0.7mm, F.Cu at (190.3, 136.7)
- added J11: Conn_01x01_Socket, TestPoint:TestPoint_THTPad_D1.5mm_Drill0.7mm, F.Cu at (189.3, 76.7)
- added J6: Conn_01x01_Socket, TestPoint:TestPoint_THTPad_D1.5mm_Drill0.7mm, F.Cu at (190.3, 131.3)
- added J7: Conn_01x01_Socket, TestPoint:TestPoint_THTPad_D1.5mm_Drill0.7mm, F.Cu at (189.1, 71.0)
- added J8: Conn_01x01_Socket, TestPoint:TestPoint_THTPad_D1.5mm_Drill0.7mm, F.Cu at (190.4, 142.4)
- added J9: Conn_01x01_Socket, TestPoint:TestPoint_THTPad_D1.5mm_Drill0.7mm, F.Cu at (189.1, 65.4)
- added TP10: TestPoint_Flag, TestPoint:TestPoint_Pad_D1.5mm, F.Cu at (130.9, 129.8)
- added TP11: TestPoint_Flag, TestPoint:TestPoint_Pad_D1.5mm, F.Cu at (150.6, 113.1)
- added TP12: TestPoint_Flag, TestPoint:TestPoint_Pad_D1.5mm, F.Cu at (97.6, 130.3)
- added TP13: TestPoint_Flag, TestPoint:TestPoint_Pad_D1.5mm, F.Cu at (81.8, 123.0)
- added TP14: TestPoint_Flag, TestPoint:TestPoint_Pad_D1.5mm, F.Cu at (110.8, 113.8)
- added TP15: TestPoint_Flag, TestPoint:TestPoint_Pad_D1.5mm, F.Cu at (133.4, 134.3)
- added TP16: TestPoint_Flag, TestPoint:TestPoint_Pad_D1.5mm, F.Cu at (130.5, 114.1)
- added TP17: TestPoint_Flag, TestPoint:TestPoint_Pad_D1.5mm, F.Cu at (112.2, 131.6)
- added TP18: TestPoint_Flag, TestPoint:TestPoint_Pad_D1.5mm, F.Cu at (167.6, 114.1)
- added TP19: TestPoint_Flag, TestPoint:TestPoint_Pad_D1.5mm, F.Cu at (184.9, 89.7)
- added TP2: TestPoint_Flag, TestPoint:TestPoint_Pad_D1.5mm, F.Cu at (187.4, 104.0)
- added TP20: TestPoint_Flag, TestPoint:TestPoint_Pad_D1.5mm, F.Cu at (118.8, 66.3)
- added TP21: TestPoint_Flag, TestPoint:TestPoint_Pad_D1.5mm, F.Cu at (179.0, 80.0)
- added TP22: TestPoint_Flag, TestPoint:TestPoint_Pad_D1.5mm, F.Cu at (137.4, 66.2)
- added TP23: TestPoint_Flag, TestPoint:TestPoint_Pad_D1.5mm, F.Cu at (162.4, 86.6)
- added TP24: TestPoint_Flag, TestPoint:TestPoint_Pad_D1.5mm, F.Cu at (158.1, 68.5)
- added TP3: TestPoint_Flag, TestPoint:TestPoint_Pad_D1.5mm, F.Cu at (253.5, 90.2)
- added TP4: TestPoint_Flag, TestPoint:TestPoint_Pad_D1.5mm, F.Cu at (252.0, 105.0)
- added TP5: TestPoint_Flag, TestPoint:TestPoint_Pad_D1.5mm, F.Cu at (225.7, 119.0)
- added TP6: TestPoint_Flag, TestPoint:TestPoint_Pad_D1.5mm, F.Cu at (220.3, 119.0)
- added TP7: TestPoint_Flag, TestPoint:TestPoint_Pad_D1.5mm, F.Cu at (209.6, 91.3)
- added TP8: TestPoint_Flag, TestPoint:TestPoint_Pad_D1.5mm, F.Cu at (206.2, 113.5)
- added TP9: TestPoint_Flag, TestPoint:TestPoint_Pad_D1.5mm, F.Cu at (187.4, 114.1)
- added U7: ~, Custom_parts:BreadBoard Space, F.Cu at (232.5, 131.4)
- added U8: ~, Custom_parts:BreadBoard Space, F.Cu at (85.6, 69.2)
- added U9: ~, Custom_parts:BreadBoard Space, F.Cu at (232.3, 69.1)
- moved TP1 140.3 mm to (99.4, 101.5)
- moved J3 1.39 mm to (252.9, 98.9)
- moved R9 1.00 mm to (147.1, 131.0)
- moved R7 0.75 mm to (147.1, 137.0)
- moved J1 0.43 mm to (75.4, 95.7)
- moved J2 0.40 mm to (75.4, 112.2)
Connections:
- TP1 pad 1: unconnected-(TP1-Pad1) -> /Mic Amp/Mic_Amp_Out
Routing:
- net (no net): track 0.00 -> 884.8 mm
- net -15V: track 428.7 -> 465.2 mm, vias 7 -> 9
- net +15V: track 439.9 -> 455.6 mm
- net Net-(Q1-S): track 27.3 -> 37.0 mm, vias 0 -> 1
- net Net-(Q1-G): track 9.10 -> 16.1 mm
- net Net-(U2D--): track 33.1 -> 39.8 mm
- net Net-(U2B-+): track 17.8 -> 24.1 mm
- net Net-(U2C-+): track 17.4 -> 23.3 mm
- net Net-(U2B--): track 36.6 -> 42.2 mm
- net Net-(U2A-+): track 16.4 -> 21.9 mm
- net Net-(D1-K): track 27.3 -> 32.8 mm
- net Net-(U2A--): track 46.4 -> 51.9 mm
- net Net-(U2D-+): track 17.1 -> 22.6 mm
- net /Shelving Filter/Shelving_Filter_Out: track 36.8 -> 42.2 mm
- net /Peak Limiter/Peak_Limit_in: track 7.96 -> 13.1 mm
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Other:
- board text added: "+15V"
- board text added: "-15V"
- board text added: "GND"
- board text added: "Mic_Amp_Gain_Adjust"
- board text added: "Out+"
- board text added: "Out-"
- board text added: "SV_Gain_Adjust"
- board text added: "SV_Select"
- board text added: "Shelf_Bass_Adjust"
- board text added: "Shelf_Select"
- board text added: "Shelf_Treble_Adjust"
- board text added: "in+"
- board text added: "in-"
- board text removed: "Shelving Filter"
- board text removed: "State Variable"
