File: ECET 318/ECET_318_Project/Peak_Limiter.kicad_sch (KiCad schematic)
At the start: 21 parts, among them Q1 2N3819, U6 TL081, U7 TL081, U8 TL081

Commit message: Mostly finished Layout and change U5 to TL084
Parts:
- removed C22: Cdec6, Capacitor_THT:C_Disc_D3.0mm_W1.6mm_P2.50mm, symbol Device:C
- removed C23: Cdec5, Capacitor_THT:C_Disc_D3.0mm_W1.6mm_P2.50mm, symbol Device:C
- removed C24: Cdec7, Capacitor_THT:C_Disc_D3.0mm_W1.6mm_P2.50mm, symbol Device:C
- removed C25: Cdec8, Capacitor_THT:C_Disc_D3.0mm_W1.6mm_P2.50mm, symbol Device:C
- removed C26: Cdec3, Capacitor_THT:C_Disc_D3.0mm_W1.6mm_P2.50mm, symbol Device:C
- removed C27: Cdec4, Capacitor_THT:C_Disc_D3.0mm_W1.6mm_P2.50mm, symbol Device:C
- removed U6, U7, U8: TL081, Package_DIP:CERDIP-8_W7.62mm_SideBrazed_LongPads_Socket, symbol Custom_parts:TL081
- added C30: Cdec6, Capacitor_THT:C_Disc_D3.0mm_W1.6mm_P2.50mm, symbol Device:C
- added C31: Cdec5, Capacitor_THT:C_Disc_D3.0mm_W1.6mm_P2.50mm, symbol Device:C
- added U5: TL084, Package_DIP:CERDIP-14_W7.62mm_SideBrazed_LongPads_Socket, symbol Amplifier_Operational:TL084
- C21: footprint Capacitor_THT:CP_Radial_D10.0mm_P5.00mm -> Capacitor_THT:C_Disc_D3.0mm_W1.6mm_P2.50mm
- D1: footprint Diode_THT:D_5W_P12.70mm_Horizontal -> Diode_THT:D_DO-34_SOD68_P7.62mm_Horizontal
Connections:
- net +15V: now also C30.1, U5.4 (V+)
- net -15V: now also C31.1, U5.11 (V-)
- net GND: now also C30.2, C31.2, U5.10 (+), U5.12 (+)
- net Peak_Limit_Out+: now also U5.1, U5.5 (+)
- net Peak_Limit_Out-: now also U5.8
- net at R35.2, R36.1: now also U5.9 (-)
- net at C21.1, D1.1 (K), R31.2: now also U5.6 (-)
- net at Q1.3 (S), R30.2: now also U5.3 (+)
- net at R33.1, R34.2: now also U5.2 (-)
- net at D1.2 (A): now also U5.7
- new net: U5.13 (-), U5.14

Commit message: Added Breadboard Space and Test Points
Parts:
- added TP3, TP4, TP5, TP6, TP7, TP8: TestPoint_Flag, TestPoint:TestPoint_Pad_D1.5mm, symbol Connector:TestPoint_Flag
Connections:
- net Peak_Limit_Out+: now also TP3.1
- net Peak_Limit_Out-: now also TP4.1
- net at Q1.2 (G), R31.1, R32.2: now also TP8.1
- net at C21.1, D1.1 (K), R31.2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: now also TP5.1
- net at R28.2, R29.2, R30.1: now also TP7.1
- net at Q1.3 (S), R30.2, U5.3 (+): now also TP6.1
