File: Power_Amplifier_Board/Class_D_IC.kicad_sch (KiCad schematic)
At the start: 0 parts

Commit message: Updated Schematic and initial layout of combined board
Parts:
- added C2, C7: C, symbol Device:C
- added U4: ~, Package_DIP:CERDIP-20_W7.62mm_SideBrazed_LongPads_Socket, symbol Custom_Parts:TPA3122
Connections:
- new net: C7.2, U4.4 (Lin)
- new net: C2.2, U4.5 (Rin)
- new net Class_D_IC_in_+: C7.1
- new net Class_D_IC_in_-: C2.1
