File: Signal_Processing_Board/Signal_Processing_Board.kicad_pcb (KiCad board)
At the start: 2 copper layers, 191 x 86.2 mm, 114 parts, among them J1 Screw_Terminal_01x02, J10 Conn_01x01_Socket, J11 Conn_01x01_Socket, J2 Screw_Terminal_01x03, J3 Screw_Terminal_01x02, J6 Conn_01x01_Socket, J7 Conn_01x01_Socket, J8 Conn_01x01_Socket, J9 Conn_01x01_Socket, Q1 2N3819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

Commit message: Roughly Finalized Signal processing board
Parts:
- added H1: MountingHole, MountingHole:MountingHole_3.2mm_M3_ISO7380_Pad, F.Cu at (73.8, 66.0)
- added H2: MountingHole, MountingHole:MountingHole_3.2mm_M3_ISO7380_Pad, F.Cu at (254.8, 66.0)
- added H3: MountingHole, MountingHole:MountingHole_3.2mm_M3_ISO7380_Pad, F.Cu at (254.8, 142.2)
- added H4: MountingHole, MountingHole:MountingHole_3.2mm_M3_ISO7380_Pad, F.Cu at (73.8, 142.2)
- added J12: Conn_01x01_Socket, TestPoint:TestPoint_THTPad_D1.5mm_Drill0.7mm, F.Cu at (73.8, 74.2)
- added J13: Conn_01x01_Socket, TestPoint:TestPoint_THTPad_D1.5mm_Drill0.7mm, F.Cu at (73.8, 79.8)
- added J14: Conn_01x01_Socket, TestPoint:TestPoint_THTPad_D1.5mm_Drill0.7mm, F.Cu at (73.8, 85.2)
- U7, U9: footprint Custom_parts:BreadBoard Space -> Custom_parts:BreadBoard Space XL
- moved C29 24.1 mm to (99.8, 144.0), turned to 90 degrees
- moved C28 7.94 mm to (86.5, 144.0), turned to 90 degrees
- moved J11 2.03 mm to (189.2, 78.8)
- moved J7 2.03 mm to (189.1, 73.1)
- moved J9 2.03 mm to (189.1, 67.4)
- moved U8 1.56 mm to (86.6, 70.4)
- moved C1 1.35 mm to (99.2, 97.0)
- moved C2 1.35 mm to (87.8, 106.2)
- moved R1 1.35 mm to (82.8, 99.5)
- moved R2 1.35 mm to (82.8, 97.0)
- moved RV4 1.35 mm to (91.5, 86.0)
- moved U1 1.35 mm to (95.3, 102.1)
- moved J1 1.25 mm to (75.5, 97.0)
- moved TP1 1.06 mm to (99.8, 102.5)
- moved U7 0.24 mm to (232.2, 131.4)
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Routing:
- net (no net): track 884.8 -> 762.8 mm, vias 0 -> 8
- net +15V: track 455.6 -> 510.3 mm, vias 5 -> 6
- net -15V: track 465.2 -> 492.0 mm
- net /Mic Amp/Mic_Amp_Out: track 198.7 -> 203.5 mm
- net Net-(R16-Pad2): track 62.4 -> 58.7 mm
- net /Peak Limiter/Peak_Limit_Out-: track 34.5 -> 32.3 mm
- net Net-(U3A--): track 54.7 -> 52.4 mm
- net Net-(C3-Pad2): track 19.8 -> 21.2 mm
- net Net-(C5-Pad2): track 20.0 -> 21.4 mm
- net /Mic Amp/Mic_Amp_in-: track 12.6 -> 11.8 mm
- net GND: vias 0 -> 104

Commit message: Minor updates to signal board, beginnings of power board
Routing:
- net Net-(U2D-+): track 22.6 -> 30.6 mm
- net +15V: track 510.3 -> 506.8 mm
- net -15V: track 492.0 -> 488.9 mm
- net /State Variable/State_Variable_Out: track 71.8 -> 74.1 mm
- net Net-(U3A--): track 52.4 -> 54.5 mm
- net Net-(D1-K): track 32.8 -> 34.1 mm
- net Net-(C16-Pad2): track 61.7 -> 60.4 mm
- net Net-(U2A--): track 51.9 -> 50.8 mm
- net Net-(U4C--): track 45.8 -> 44.8 mm
- net Net-(C5-Pad2): track 21.4 -> 22.4 mm
- net Net-(U2C--): track 57.4 -> 56.5 mm
- net Net-(U10B--): track 26.9 -> 26.0 mm
- net /Shelving Filter/Shelving_Filter_Out: track 42.2 -> 41.4 mm
- net Net-(C3-Pad2): track 21.2 -> 21.9 mm
- net Net-(Q1-S): track 37.0 -> 36.4 mm
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Other:
- outline, holes or cut-outs redrawn

Commit message: Minor updates to the signal processing board
Routing:
- net /State Variable/State_Variable_Out: track 74.1 -> 75.8 mm
- net GND: vias 115 -> 119
Changed lines of the file:
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@@
 	)
 	(via
+		(at 119 107)
+		(size 0.6)
+		(drill 0.3)
+		(layers "F.Cu" "B.Cu")
+		(free yes)
+		(net 2)
+	)
+	(via
 		(at 235.5 110.25)
 		(size 0.6)
@@
 	)
 	(via
+		(at 104.75 101.5)
+		(size 0.6)
+		(drill 0.3)
+		(layers "F.Cu" "B.Cu")
+		(free yes)
+		(net 2)
+	)
+	(via
 		(at 128.25 84.25)
 		(size 0.6)
@@
 	)
 	(via
+		(at 125.75 107)
+		(size 0.6)
+		(drill 0.3)
+		(layers "F.Cu" "B.Cu")
+		(free yes)
+		(net 2)
+	)
+	(via
 		(at 127.75 141)
 		(size 0.6)
@@
 	)
 	(via
+		(at 111.75 107)
+		(size 0.6)
+		(drill 0.3)
+		(layers "F.Cu" "B.Cu")
+		(free yes)
+		(net 2)
+	)
+	(via
 		(at 249 120.5)
 		(size 0.6)
@@
 	)
 	(segment
+		(start 203.25 94.503963)
+		(end 203.25 101.906036)
+		(width 0.5)
+		(layer "F.Cu")
+		(net 3)
+	)
+	(segment
 		(start 167.925 137.695)
 		(end 167.92 137.7)
@@
 	)
 	(segment
-		(start 194.496036 85.75)
-		(end 183.5 85.75)
-		(width 0.5)
-		(layer "F.Cu")
-		(net 3)
-	)
-	(segment
 		(start 167.149999 137.849999)
 		(end 167.429999 137.569999)
@@
 	)
 	(segment
+		(start 184.044418 85.75)
+		(end 194.496036 85.75)
+		(width 0.5)
+		(layer "F.Cu")
+		(net 3)
+	)
+	(segment
 		(start 121.38125 138.88125)
 		(end 121.19375 138.69375)
@@
 	)
 	(segment
+		(start 183.541814 85.541814)
+		(end 183.333629 85.333629)
+		(width 0.5)
+		(layer "F.Cu")
+		(net 3)
+	)
+	(segment
 		(start 125.83 122.04)
 		(end 125.749999 122.119999)
@@
 	)
 	(segment
-		(start 203.25 101.906036)
-		(end 203.25 94.503963)
+		(start 167.149999 137.849999)
+		(end 163.193792 141.806207)
 		(width 0.5)
 		(layer "F.Cu")
@@
 	)
 	(segment
-		(start 167.149999 137.849999)
-		(end 163.193792 141.806207)
+		(start 201.656207 105.753792)
+		(end 199.465 107.945)
 		(width 0.5)
 		(layer "F.Cu")
@@
 		(net 3)
 	)
-	(segment
-		(start 201.656207 105.753792)
-		(end 199.465 107.945)
-		(width 0.5)
-		(layer "F.Cu")
-		(net 3)
-	)
 	(via
 		(at 246.75 112.75)
@@
 	)
 	(via
-		(at 183.5 85.75)
+		(at 183.333629 85.333629)
 		(size 0.6)
 		(drill 0.3)
@@
 	)
 	(arc
-		(start 203.25 101.906036)
-		(mid 202.835786 103.988426)
-		(end 201.656207 105.753792)
-		(width 0.5)
-		(layer "F.Cu")
-		(net 3)
-	)
-	(arc
 		(start 87.75 107.125)
 		(mid 87.5892 107.933394)
@@
 	)
 	(arc
-		(start 198.343792 87.343792)
-		(mid 196.578426 86.164213)
-		(end 194.496036 85.75)
-		(width 0.5)
-		(layer "F.Cu")
-		(net 3)
-	)
-	(arc
 		(start 175.75 128.177243)
 		(mid 175.644743 128.706401)
@@
 	)
 	(arc
+		(start 203.25 101.906036)
+		(mid 202.835786 103.988426)
+		(end 201.656207 105.753792)
+		(width 0.5)
+		(layer "F.Cu")
+		(net 3)
+	)
+	(arc
 		(start 125.926568 122)
 		(mid 125.874305 122.010395)
@@
 	)
 	(arc
+		(start 183.541814 85.541814)
+		(mid 183.77241 85.695894)
+		(end 184.044418 85.75)
+		(width 0.5)
+		(layer "F.Cu")
+		(net 3)
+	)
+	(arc
+		(start 194.496036 85.75)
+		(mid 196.578426 86.164213)
+		(end 198.343792 87.343792)
+		(width 0.5)
+		(layer "F.Cu")
+		(net 3)
+	)
+	(arc
 		(start 120.882842 138.9)
 		(mid 120.621529 138.951978)
@@
 	)
 	(arc
+		(start 201.656207 90.656207)
+		(mid 202.835786 92.421572)
+		(end 203.25 94.503963)
+		(width 0.5)
+		(layer "F.Cu")
+		(net 3)
+	)
+	(arc
 		(start 120.80625 138.69375)
 		(mid 120.949646 138.479142)
@@
 	)
 	(arc
-		(start 201.656207 90.656207)
-		(mid 202.835786 92.421572)
-		(end 203.25 94.503963)
-		(width 0.5)
-		(layer "F.Cu")
-		(net 3)
-	)
-	(arc
 		(start 167.925 137.685)
 		(mid 167.93 137.687071)
@@
 	)
 	(segment
+		(start 231.38 96)
+		(end 223.49 96)
+		(width 0.5)
+		(layer "F.Cu")
+		(net 25)
+	)
+	(segment
 		(start 252.805 96.255)
 		(end 252.88 96.33)
@@
 	)
 	(segment
-		(start 231.35 95.97)
-		(end 231.875 96.495)
+		(start 247.195 86.945)
+		(end 234.38599 86.945)
 		(width 0.5)
 		(layer "F.Cu")
@@
 	)
 	(segment
-		(start 231.21 95.83)
-		(end 231.875 96.495)
-		(width 0.5)
-		(layer "F.Cu")
-		(net 25)
-	)
-	(segment
-		(start 230.082537 95.445)
-		(end 222.935 95.445)
+		(start 231.875 96.495)
+		(end 231.38 96)
 		(width 0.5)
 		(layer "F.Cu")
@@
 	(segment
 		(start 230.545 89.195)
-		(end 230.545 94.224547)
+		(end 230.545 93.284138)
 		(width 0.5)
 		(layer "F.Cu")
@@
 	)
 	(segment
-		(start 230.545 89.195)
-		(end 231.67 88.07)
+		(start 231.67 88.07)
+		(end 230.545 89.195)
 		(width 0.5)
 		(layer "F.Cu")
@@
 	)
 	(segment
-		(start 234.625 98.970304)
-		(end 234.625 104.5894)
+		(start 252.093933 91.843933)
+		(end 247.195 86.945)
 		(width 0.5)
 		(layer "F.Cu")
@@
 	)
 	(segment
-		(start 247.261871 87.011871)
-		(end 252.093933 91.843933)
+		(start 223.49 96)
+		(end 222.935 95.445)
 		(width 0.5)
 		(layer "F.Cu")
@@
 	)
 	(segment
-		(start 247.1125 86.95)
-		(end 247.028535 86.95)
+		(start 234.625 98.970304)
+		(end 234.625 104.5894)
 		(width 0.5)
 		(layer "F.Cu")
@@
 	)
 	(segment
-		(start 234.38599 86.945)
-		(end 247.016464 86.945)
-		(width 0.5)
-		(layer "F.Cu")
-		(net 25)
-	)
-	(segment
 		(start 232.525 96.495)
 		(end 231.875 96.495)
@@
 	)
 	(arc
-		(start 247.0225 86.9475)
-		(mid 247.01973 86.945649)
-		(end 247.016464 86.945)
-		(width 0.5)
-		(layer "F.Cu")
-		(net 25)
-	)
-	(arc
 		(start 233.634619 96.954619)
 		(mid 233.125521 96.614451)
@@
 	)
 	(arc
-		(start 247.261871 87.011871)
-		(mid 247.193339 86.966079)
-		(end 247.1125 86.95)
-		(width 0.5)
-		(layer "F.Cu")
-		(net 25)
-	)
-	(arc
-		(start 247.0225 86.9475)
-		(mid 247.025268 86.94935)
-		(end 247.028535 86.95)
-		(width 0.5)
-		(layer "F.Cu")
-		(net 25)
-	)
-	(arc
-		(start 231.35 95.97)
-		(mid 230.768483 95.581443)
-		(end 230.082537 95.445)
+		(start 230.545 93.284138)
+		(mid 230.890648 95.021828)
+		(end 231.875 96.495)
 		(width 0.5)
 		(layer "F.Cu")
@@
 	)
 	(arc
-		(start 230.545 94.224547)
-		(mid 230.717827 95.093412)
-		(end 231.21 95.83)
+		(start 252.093933 91.843933)
+		(mid 252.161644 91.857402)
+		(end 252.2 91.8)
 		(width 0.5)
 		(layer "F.Cu")
@@
 	)
 	(arc
-		(start 252.093933 91.843933)
-		(mid 252.161644 91.857402)
-		(end 252.2 91.8)
+		(start 252.73 96.073933)
+		(mid 252.749491 96.171925)
+		(end 252.805 96.255)
 		(width 0.5)
 		(layer "F.Cu")
@@
 		(net 25)
 	)
-	(arc
-		(start 252.73 96.073933)
-		(mid 252.749491 96.171925)
-		(end 252.805 96.255)
+	(segment
+		(start 181.75 91.275)
+		(end 181.75 90)
 		(width 0.5)
 		(layer "F.Cu")
-		(net 25)
+		(net 26)
 	)
 	(segment
@@
 	)
 	(segment
+		(start 181.75 89.5)
+		(end 181.75 88.125)
+		(width 0.5)
+		(layer "F.Cu")
+		(net 26)
+	)
+	(segment
 		(start 183.325 89.7)
 		(end 184.9 89.7)
@@
 	)
 	(segment
+		(start 181.814381 89.564381)
+		(end 181.75 89.5)
+		(width 0.5)
+		(layer "F.Cu")
+		(net 26)
+	)
+	(segment
+		(start 181.75 90)
+		(end 181.75 89.5)
+		(width 0.5)
+		(layer "F.Cu")
+		(net 26)
+	)
+	(segment
+		(start 181.814381 90)
+		(end 182.25 89.564381)
+		(width 0.5)
+		(layer "F.Cu")
+		(net 26)
+	)
+	(segment
 		(start 167.79 73.75)
 		(end 167.25 73.75)
@@
 	)
 	(segment
+		(start 182.25 89.564381)
+		(end 181.814381 89.564381)
+		(width 0.5)
+		(layer "F.Cu")
+		(net 26)
+	)
+	(segment
+		(start 182.685619 89.564381)
+		(end 182.25 89.564381)
+		(width 0.5)
+		(layer "F.Cu")
+		(net 26)
+	)
+	(segment
 		(start 166.4875 103.4875)
 		(end 166.25 103.25)
@@
 	)
 	(segment
+		(start 181.75 90)
+		(end 181.814381 90)
+		(width 0.5)
+		(layer "F.Cu")
+		(net 26)
+	)
+	(segment
 		(start 180.156207 95.843792)
 		(end 177.593792 98.406207)
@@
 		(width 0.5)
 		(layer "F.Cu")
-		(net 26)
-	)
-	(segment
-		(start 181.75 91.275)
-		(end 181.75 88.125)
-		(width 0.5)
-		(layer "F.Cu")

Commit message: Updated Schematic and initial layout of combined board
Parts:
- removed J3: Screw_Terminal_01x02, TerminalBlock_TE-Connectivity:TerminalBlock_TE_282834-2_1x02_P2.54mm_Horizontal
- added C22: Cin1, Capacitor_THT:CP_Radial_D10.0mm_P5.00mm, F.Cu at (326.2, 167.2)
- added C23: Cin2, Capacitor_THT:CP_Radial_D10.0mm_P5.00mm, F.Cu at (326.2, 178.8)
- added C24: C_amp-c_f-1, Capacitor_THT:C_Disc_D3.0mm_W1.6mm_P2.50mm, F.Cu at (380.0, 93.7)
- added C25: C_amp-c_f-2, Capacitor_THT:C_Disc_D3.0mm_W1.6mm_P2.50mm, F.Cu at (348.5, 94.5)
- added C26: Cdec25, Capacitor_THT:C_Disc_D3.0mm_W1.6mm_P2.50mm, F.Cu at (358.0, 111.0)
- added C27: Cdec26, Capacitor_THT:C_Disc_D3.0mm_W1.6mm_P2.50mm, F.Cu at (348.5, 123.8)
- added C32: Cdec21, Capacitor_THT:C_Disc_D3.0mm_W1.6mm_P2.50mm, F.Cu at (389.8, 110.4)
- added C33: Cdec22, Capacitor_THT:C_Disc_D3.0mm_W1.6mm_P2.50mm, F.Cu at (380.0, 123.2)
- added C34: Cdec23, Capacitor_THT:C_Disc_D3.0mm_W1.6mm_P2.50mm, F.Cu at (368.0, 76.0)
- added C35: Cdec24, Capacitor_THT:C_Disc_D3.0mm_W1.6mm_P2.50mm, F.Cu at (394.5, 76.0)
- added C36: Cdec27, Capacitor_THT:C_Disc_D3.0mm_W1.6mm_P2.50mm, F.Cu at (336.8, 76.0)
- added C37: Cdec28, Capacitor_THT:C_Disc_D3.0mm_W1.6mm_P2.50mm, F.Cu at (362.8, 76.0)
- added J15: Screw_Terminal_01x03, TerminalBlock_TE-Connectivity:TerminalBlock_TE_282834-3_1x03_P2.54mm_Horizontal, F.Cu at (323.7, 77.8)
- added J16: Screw_Terminal_01x03, TerminalBlock_TE-Connectivity:TerminalBlock_TE_282834-3_1x03_P2.54mm_Horizontal, F.Cu at (401.5, 96.7)
- added J17: ~, Connector_PinHeader_2.54mm:PinHeader_1x02_P2.54mm_Vertical, F.Cu at (209.0, 92.5)
- added Q2: Q_amp-c-1, Package_TO_SOT_THT:TO-220-3_Vertical, F.Cu at (372.5, 75.1)
- added Q3: Q_amp-c-2, Package_TO_SOT_THT:TO-220-3_Vertical, F.Cu at (385.0, 75.1)
- added Q4: Q_amp-c-3, Package_TO_SOT_THT:TO-220-3_Vertical, F.Cu at (341.2, 75.5)
- added Q5: Q_amp-c-4, Package_TO_SOT_THT:TO-220-3_Vertical, F.Cu at (353.3, 75.5)
- added R39: R_amp-c_2, Resistor_THT:R_Axial_DIN0207_L6.3mm_D2.5mm_P10.16mm_Horizontal, F.Cu at (378.0, 89.9)
- added R40: R_amp-c_1, Resistor_THT:R_Axial_DIN0207_L6.3mm_D2.5mm_P10.16mm_Horizontal, F.Cu at (371.2, 79.8)
- added R41: R_amp-c_3, Resistor_THT:R_Axial_DIN0207_L6.3mm_D2.5mm_P10.16mm_Horizontal, F.Cu at (384.5, 89.9)
- added R42: R_amp-c_4, Resistor_THT:R_Axial_DIN0207_L6.3mm_D2.5mm_P10.16mm_Horizontal, F.Cu at (391.0, 89.9)
- added R43: R_amp-c_f-1, Resistor_THT:R_Axial_DIN0207_L6.3mm_D2.5mm_P10.16mm_Horizontal, F.Cu at (376.2, 99.9)
- added R44: R_amp-c_i-1, Resistor_THT:R_Axial_DIN0207_L6.3mm_D2.5mm_P10.16mm_Horizontal, F.Cu at (371.5, 116.8)
- added R45: R_amp-c_5, Resistor_THT:R_Axial_DIN0207_L6.3mm_D2.5mm_P10.16mm_Horizontal, F.Cu at (340.0, 80.7)
- added R46: R_amp-c_6, Resistor_THT:R_Axial_DIN0207_L6.3mm_D2.5mm_P10.16mm_Horizontal, F.Cu at (346.5, 90.8)
- added R47: R_amp-c_7, Resistor_THT:R_Axial_DIN0207_L6.3mm_D2.5mm_P10.16mm_Horizontal, F.Cu at (353.0, 90.8)
- added R48: R_amp-c_8, Resistor_THT:R_Axial_DIN0207_L6.3mm_D2.5mm_P10.16mm_Horizontal, F.Cu at (359.5, 90.8)
- added R49: R_amp-c_i-2, Resistor_THT:R_Axial_DIN0207_L6.3mm_D2.5mm_P10.16mm_Horizontal, F.Cu at (340.5, 107.4)
- added R50: R_amp-c_f-2, Resistor_THT:R_Axial_DIN0207_L6.3mm_D2.5mm_P10.16mm_Horizontal, F.Cu at (344.7, 100.5)
- added R51: R_amp-c_in-1, Resistor_THT:R_Axial_DIN0207_L6.3mm_D2.5mm_P10.16mm_Horizontal, F.Cu at (334.5, 107.4)
- added U11: U_amp-c_1, Package_DIP:CERDIP-8_W7.62mm_SideBrazed_LongPads_Socket, F.Cu at (377.4, 107.9)
- added U12: U_amp-c_2, Package_DIP:CERDIP-8_W7.62mm_SideBrazed_LongPads_Socket, F.Cu at (345.9, 108.4)
- moved TP3 51.9 mm to (201.6, 88.8)
- moved TP4 51.0 mm to (201.1, 106.8)
- moved R25 47.2 mm to (128.9, 95.3)
- moved R34 47.2 mm to (175.8, 89.0)
- moved C11 47.2 mm to (66.3, 124.3)
- moved R12 47.2 mm to (104.3, 106.6)
- moved R13 47.2 mm to (124.7, 113.9)
- moved R8 47.2 mm to (89.8, 106.6)
- moved R9 47.2 mm to (99.9, 130.8)
- moved TP10 47.2 mm to (83.7, 129.6)
- moved TP15 47.2 mm to (86.2, 134.1)
- moved TP22 47.2 mm to (90.2, 66.0)
- moved TP23 47.2 mm to (115.2, 86.4)
- moved C10 47.2 mm to (45.4, 131.6)
- moved C7 47.2 mm to (55.6, 131.6)
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Routing:
- net -HV: track 0.00 -> 151.7 mm
- net +HV: track 0.00 -> 112.9 mm
- net /Class_B_Discrete/Class_B_Discrete_Out_-: track 0.00 -> 104.0 mm
- net /Class_B_Discrete/Class_B_Discrete_Out_+: track 0.00 -> 71.8 mm
- net /Class_B_Discrete/Class_B_Discrete_in: track 0.00 -> 57.8 mm
- net Net-(U11A-Out): track 0.00 -> 46.6 mm
- net Net-(U12A-Out): track 0.00 -> 44.7 mm
- net Net-(U11A--): track 0.00 -> 24.0 mm
- net Net-(U12A--): track 0.00 -> 23.1 mm
- net Net-(Q4-G): track 0.00 -> 22.7 mm, vias 0 -> 1
- net Net-(Q2-G): track 0.00 -> 22.4 mm, vias 0 -> 1
- net Net-(Q5-G): track 0.00 -> 18.1 mm
- net Net-(Q3-G): track 0.00 -> 17.7 mm
- net /Peak Limiter/Peak_Limit_Out-: track 32.3 -> 20.5 mm
- net /Peak Limiter/Peak_Limit_Out+: track 62.6 -> 57.0 mm
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- removed copper zone on B.Cu, net GND
- removed copper zone on F.Cu, net GND
Other:
- board size 191 x 86.2 mm -> 186 x 86.2 mm
- board text added: "+HV"
- board text added: "-HV"
- board text added: "PGN"
- board text removed: "Out+"
- board text removed: "Out-"

Commit message: First semi-finalized layout done
Parts:
- added H5: MountingHole, MountingHole:MountingHole_3.2mm_M3_ISO7380_Pad, F.Cu at (264.0, 103.5)
- added H6: MountingHole, MountingHole:MountingHole_3.2mm_M3_ISO7380_Pad, F.Cu at (264.0, 180.2)
- added H7: MountingHole, MountingHole:MountingHole_3.2mm_M3_ISO7380_Pad, F.Cu at (349.8, 103.5)
- added H8: MountingHole, MountingHole:MountingHole_3.2mm_M3_ISO7380_Pad, F.Cu at (349.8, 180.2)
- added J18: Conn_01x01_Socket, TestPoint:TestPoint_THTPad_D1.5mm_Drill0.7mm, F.Cu at (274.8, 171.2)
- added J19: Conn_01x01_Socket, TestPoint:TestPoint_THTPad_D1.5mm_Drill0.7mm, F.Cu at (274.8, 176.8)
- added J3: Conn_01x01_Socket, TestPoint:TestPoint_THTPad_D1.5mm_Drill0.7mm, F.Cu at (274.8, 165.5)
- added U13: ~, Custom_parts:BreadBoard Space XL, F.Cu at (321.9, 169.2)
- C22: value Cin1 -> Cin3
- C23: value Cin2 -> Cin4
- moved C23 72.6 mm to (272.9, 129.5)
- moved C22 70.7 mm to (277.8, 115.8), turned to 180 degrees
- moved J11 67.0 mm to (197.2, 116.6)
- moved J7 67.0 mm to (197.1, 110.9)
- moved J9 67.0 mm to (197.1, 105.2)
- moved H4 66.7 mm to (81.2, 180.2)
- moved R25 66.6 mm to (183.6, 133.3)
- moved R12 66.6 mm to (159.0, 144.6)
- moved R19 66.6 mm to (112.5, 135.8)
- moved R34 66.6 mm to (230.5, 127.0)
- moved R8 66.6 mm to (144.5, 144.6)
- moved R9 66.6 mm to (154.6, 168.8)
- moved TP10 66.6 mm to (138.4, 167.6)
- moved TP15 66.6 mm to (140.9, 172.1)
- moved TP22 66.6 mm to (144.9, 104.0)
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Connections:
- C22 pad 2: GND -> GNDPWR
- C23 pad 2: GND -> GNDPWR
- J15 pad 2: GND -> GNDPWR
Routing:
- net (no net): track 762.6 -> 1098.2 mm
- net -HV: track 151.7 -> 315.1 mm
- net +HV: track 112.9 -> 245.2 mm, vias 0 -> 6
- net GND: track 19.1 -> 94.4 mm, vias 102 -> 125
- net /Class_B_Discrete/Class_B_Discrete_in: track 57.8 -> 87.9 mm, vias 0 -> 1
- net /Class_B_Discrete/Class_B_Discrete_Out_-: track 104.0 -> 109.5 mm, vias 0 -> 9
- net Net-(Q2-G): track 22.4 -> 25.7 mm
- net -15V: track 489.2 -> 492.2 mm
- net Net-(Q4-G): track 22.7 -> 25.5 mm
- net /Class_B_Discrete/Class_B_Discrete_Out_+: track 71.8 -> 70.5 mm
- net +15V: track 506.8 -> 508.0 mm
- net Net-(U2D-+): track 30.6 -> 31.7 mm
- net Net-(U11A-Out): track 46.6 -> 45.8 mm
- net Net-(U12A-Out): track 44.7 -> 44.0 mm
- net Net-(U2C-+): track 22.8 -> 22.2 mm
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- added copper zone on B.Cu, net GND
- added copper zone on F.Cu, net GND
- added copper zone on B.Cu, net GNDPWR
- added copper zone on F.Cu, net GNDPWR
Other:
- board size 186 x 86.2 mm -> 278.5 x 86.8 mm
- board text added: "Out+"
- board text added: "Out-"
- board text added: "PGND"
- board text removed: "PGN"
