File: Signal_Processing_Board/Signal_Processing_Board.kicad_pcb (KiCad board)
At the start: 2 copper layers, 278.5 x 86.8 mm, 162 parts, among them J1 Screw_Terminal_01x02, J10 Conn_01x01_Socket, J11 Conn_01x01_Socket, J12 Conn_01x01_Socket, J13 Conn_01x01_Socket, J14 Conn_01x01_Socket, J15 Screw_Terminal_01x03, J16 Screw_Terminal_01x03, J18 Conn_01x01_Socket, J19 Conn_01x01_Socket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

Commit message: First ordered version of Board
Parts:
- added TP25: TestPoint_Flag, TestPoint:TestPoint_Pad_D1.5mm, F.Cu at (349.5, 119.8)
- added TP26: TestPoint_Flag, TestPoint:TestPoint_Pad_D1.5mm, F.Cu at (347.8, 133.8)
- added TP27: TestPoint_Flag, TestPoint:TestPoint_Pad_D1.5mm, F.Cu at (289.5, 131.0)
- added TP28: TestPoint_Flag, TestPoint:TestPoint_Pad_D1.5mm, F.Cu at (310.5, 137.2)
- added TP29: TestPoint_Flag, TestPoint:TestPoint_Pad_D1.5mm, F.Cu at (317.2, 133.8)
- added TP30: TestPoint_Flag, TestPoint:TestPoint_Pad_D1.5mm, F.Cu at (342.2, 136.5)
- C22: value Cin3 -> Cin1
- C23: value Cin4 -> Cin2
- moved Q4 0.31 mm to (290.2, 102.2)
- moved Q5 0.31 mm to (302.3, 102.2)
Connections:
- J18 pad 1: GND -> GNDPWR
Routing:
- net GND: track 94.4 -> 218.2 mm
- net +HV: track 245.2 -> 236.0 mm, vias 6 -> 2
- net Net-(U12A--): track 22.8 -> 26.2 mm
- net Net-(U11A--): track 23.6 -> 26.9 mm
- net /Class_B_Discrete/Class_B_Discrete_Out_-: track 109.5 -> 106.5 mm, vias 9 -> 2
- net +15V: track 508.0 -> 509.1 mm
- net Net-(U12A-Out): track 44.0 -> 45.0 mm
- net Net-(U4D--): track 27.3 -> 27.9 mm
- net Net-(D1-K): track 34.6 -> 35.2 mm
- net GNDPWR: vias 77 -> 74
Other:
- board text added: "ECET 318 Board V1"

Commit message: Final version of the board, updated with lessons from first version
Parts:
- added C38: Cdec29, Capacitor_THT:CP_Radial_D10.0mm_P5.00mm, F.Cu at (358.0, 114.6)
- added C39: Cdec30, Capacitor_THT:CP_Radial_D10.0mm_P5.00mm, F.Cu at (318.3, 116.0)
- added C40: Cdec31, Capacitor_THT:CP_Radial_D10.0mm_P5.00mm, F.Cu at (318.3, 101.5)
- added C41: Cdec32, Capacitor_THT:CP_Radial_D10.0mm_P5.00mm, F.Cu at (277.6, 114.1)
- Q1: footprint Package_TO_SOT_THT:TO-92 -> Package_TO_SOT_THT:TO-92_Inline
- moved C22 19.8 mm to (277.6, 135.5)
- moved J16 12.1 mm to (361.3, 124.0)
- moved H8 12.0 mm to (361.7, 180.2)
- moved H7 11.9 mm to (361.7, 103.5)
- moved C24 7.79 mm to (336.8, 120.7)
- moved C32 7.79 mm to (346.5, 137.4)
- moved C33 7.79 mm to (336.8, 150.2)
- moved C34 7.79 mm to (324.8, 103.0)
- moved C35 7.79 mm to (351.3, 103.0)
- moved Q2 7.79 mm to (329.2, 102.1)
- moved Q3 7.79 mm to (341.8, 102.1)
- moved R39 7.79 mm to (334.8, 116.9)
- moved R40 7.79 mm to (328.0, 106.8)
- moved R41 7.79 mm to (341.3, 116.9)
- moved R42 7.79 mm to (347.8, 116.9)
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Connections:
- C19 pad 2: -15V -> +15V
- C20 pad 2: +15V -> -15V
- C23 pad 1: -HV -> GNDPWR
- C23 pad 2: GNDPWR -> -HV
- Q1 pad 1: GND -> Net-(Q1-S)
- Q1 pad 2: Net-(Q1-G) -> GND
- Q1 pad 3: Net-(Q1-S) -> Net-(Q1-G)
- U4 pad 11: +15V -> -15V
- U4 pad 4: -15V -> +15V
Routing:
- net GND: track 218.2 -> 294.9 mm, vias 125 -> 126
- net -HV: track 315.5 -> 368.7 mm
- net +HV: track 236.0 -> 256.6 mm
- net /Class_B_Discrete/Class_B_Discrete_Out_-: track 106.5 -> 119.1 mm
- net -15V: track 492.2 -> 503.4 mm, vias 9 -> 11
- net /Class_B_Discrete/Class_B_Discrete_in: track 87.9 -> 95.9 mm
- net /Class_B_Discrete/Class_B_Discrete_Out_+: track 70.0 -> 77.8 mm, vias 0 -> 2
- net Net-(U3A--): track 54.6 -> 59.7 mm
- net Net-(Q1-S): track 36.4 -> 39.0 mm, vias 1 -> 2
- net Net-(RV4-Pad2): track 11.3 -> 13.9 mm
- net Net-(R25-Pad2): track 12.0 -> 14.5 mm
- net Net-(Q1-G): track 17.0 -> 18.7 mm
- net +15V: track 509.1 -> 510.4 mm
- net Net-(U12A-Out): track 45.0 -> 45.7 mm
- net Net-(U4D--): track 27.9 -> 28.6 mm
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Other:
- board size 278.5 x 86.8 mm -> 290.5 x 86.8 mm
