File: Signal_Processing_Board/Shelving_Filter.kicad_sch (KiCad schematic)
At the start: 37 parts, among them U2 TL084, U3 TL081

Commit message: Updated file structure and added PDF of schematic
Other:
- note added: "Op-Amp Power"
- note added: "Shelving Filter"
- moved on the sheet: C11, C12, C13, C14, U2E, U3B
